File: pcb/CoCoSDCExt.sch (EAGLE design)
At the start: 49 parts, among them IC1 AM29F040J, IC10 YAC512-M, IC14 TL974, IC15 TL974, IC2 XC9572XLVQG64, IC3 AS6C4008SIN, IC9 YMF262-M, X1 EXPANSION_PORT_COCO, X2 EXPANSION_PORT_COCOS

Commit message: nearly routed
Connections:
- removed net !CE_SN: IC2.FB2MC11-I/O/GTS2
- removed net !CE_YM: IC2.FB2MC3
- removed net !RESET_YM: IC2.FB2MC4
- removed net !WE_SN: IC2.FB2MC14-I/O/GTS1
- removed net A0_YM: IC2.FB4MC17
- removed net BD0: IC2.FB2MC10
- removed net BD1: IC2.FB2MC12
- removed net BD2: IC2.FB2MC15
- removed net BD3: IC2.FB1MC2
- removed net BD4: IC2.FB1MC3
- removed net BD5: IC2.FB1MC4
- removed net BD6: IC2.FB1MC8
- removed net BD7: IC2.FB1MC5
- removed net CH2: IC2.FB2MC2
- removed net CLK_SN: IC2.FB1MC6
- removed net CLK_YM: IC2.FB4MC15
- removed net READY: IC2.FB2MC17
- new net !CE_FLASH: IC1G$1.!CE, IC2.FB2MC11-I/O/GTS2
- new net !CE_RAM: IC2.FB4MC4, IC3A.!CE
- net !CTS: now also IC2.FB1MC17; no longer IC1G$1.!OE
- net !RESET: now also IC2.FB2MC12; no longer IC2.FB1MC10-I/O/GCK2
- net !SCS: now also IC2.FB1MC12; no longer IC2.FB4MC11
- net !SLENB: now also IC2.FB3MC8; no longer IC2.FB4MC14
- net !WE: now also IC2.FB4MC10, IC3A.!WE; no longer IC2.FB3MC16
- net +5V: now also IC3P.VCC@1
- net A0: now also IC2.FB2MC14-I/O/GTS1, IC3A.A7; no longer IC2.FB3MC4
- net A1: now also IC2.FB2MC10, IC3A.A6; no longer IC2.FB3MC14
- net A10: now also IC2.FB4MC6, IC3A.A15
- net A11: now also IC2.FB4MC14, IC3A.A17
- net A12: now also IC2.FB1MC14-I/O/GCK3, IC3A.A12
- net A13: now also IC2.FB2MC4, IC3A.A18; no longer IC2.FB3MC11
- net A14: now also IC2.FB3MC5; no longer IC2.FB4MC6
- net A15: now also IC2.FB3MC9; no longer IC2.FB3MC6
- net A2: now also IC2.FB2MC9-I/O/GSR, IC3A.A5; no longer IC2.FB3MC17
- net A3: now also IC2.FB2MC8, IC3A.A4; no longer IC2.FB3MC12
- net A4: now also IC2.FB2MC6, IC3A.A3; no longer IC2.FB4MC2
- net A5: now also IC2.FB2MC5, IC3A.A2; no longer IC2.FB4MC8
- net A6: now also IC2.FB2MC2, IC3A.A1
- net A7: now also IC2.FB2MC3, IC3A.A0
- net A8: now also IC2.FB1MC10, IC3A.A8
- net A9: now also IC2.FB4MC12, IC3A.A13
- net BA14: now also IC2.FB4MC17, IC3A.A9; no longer IC2.FB3MC15
- net BA15: now also IC2.FB1MC15, IC3A.A14; no longer IC2.FB4MC4
- net BA16: now also IC2.FB3MC2, IC3A.A16; no longer IC2.FB4MC3
- net BA17: now also IC2.FB4MC15, IC3A.A11; no longer IC2.FB3MC10
- net BA18: now also IC2.FB4MC11, IC3A.A10; no longer IC2.FB4MC5
- net D0: now also IC2.FB1MC4, IC3A.D3; no longer IC2.FB1MC10
- net D1: now also IC2.FB1MC3, IC3A.D2; no longer IC2.FB1MC15
- net D2: now also IC2.FB1MC8, IC3A.D4; no longer IC2.FB1MC17
- net D3: now also IC2.FB1MC6, IC3A.D1; no longer IC2.FB3MC2
- net D4: now also IC2.FB1MC5, IC3A.D5; no longer IC2.FB1MC12
- net D5: now also IC2.FB1MC2, IC3A.D0; no longer IC2.FB3MC5
- net D6: now also IC2.FB2MC17, IC3A.D6; no longer IC2.FB3MC8
- net D7: now also IC2.FB2MC15, IC3A.D7; no longer IC2.FB3MC9
- net E: now also IC2.FB1MC9-I/O/GCK1; no longer IC2.FB1MC14-I/O/GCK3
- net GND: now also IC1G$1.!OE, IC3A.!OE, IC3P.GND@1; no longer IC1G$1.!CE
- net R/!W: now also IC2.FB1MC10-I/O/GCK2; no longer IC2.FB3MC3
Other:
- moved on the sheet: IC3
